File: Pro_Smolcro/Pro_Smolcro.kicad_pcb (KiCad board)
At the start: 2 copper layers, 18 x 33 mm, 32 parts, among them J1 SHOU HAN TYPE-C 16PIN 2MD(073), J2 Conn_01x05, J3 Conn_01x13, J4 Conn_01x13, SW1 SW_Push, SW2 SW_Push, U1 RP2040, U3 W25Q128JVS, U4 TLV75733PDBV, Y1 ABM8-272-T3

Commit message: finished the layout
Parts:
- removed R5: 10k, Resistor_SMD:R_0402_1005Metric
- removed R6: 1k, Resistor_SMD:R_0402_1005Metric
- removed SW1, SW2: SW_Push, MyKeebLib:SW_TS-1088-AR02016
- added D4: LED, LED_SMD:LED_0402_1005Metric, F.Cu at (125.5, 88.2)
- added R8: 68R, Resistor_SMD:R_0402_1005Metric, F.Cu at (125.5, 90.3)
- added TP4: TestPoint, TestPoint:TestPoint_Pad_1.0x1.0mm, B.Cu at (127.8, 99.1)
- added TP5: TestPoint, TestPoint:TestPoint_Pad_1.0x1.0mm, B.Cu at (127.8, 97.0)
- moved C4 12.2 mm to (126.2, 92.7)
- moved U3 1.14 mm to (128.4, 97.9), turned to 90 degrees
- moved C6 0.56 mm to (126.4, 104.2)
- moved Y1 0.40 mm to (127.9, 113.4)
- moved C10 0.28 mm to (134.4, 112.5)
- moved C9 0.28 mm to (133.3, 112.5)
- moved C2 0.11 mm to (136.1, 98.7)
- moved C12 0.05 mm to (136.8, 101.0)
- moved C13 0.05 mm to (136.8, 104.3)
Connections:
- U4 pad 4: unconnected-(U4-NC-Pad4) -> GND
Routing:
- net GP11: track 0.00 -> 35.3 mm, vias 0 -> 1
- net GP10: track 0.00 -> 28.6 mm, vias 0 -> 1
- net RST: track 0.00 -> 27.1 mm, vias 0 -> 1
- net GP0: track 0.00 -> 20.1 mm, vias 0 -> 1
- net GP1: track 0.00 -> 18.3 mm, vias 0 -> 1
- net 3V3: track 35.5 -> 50.2 mm
- net D1: track 17.7 -> 3.24 mm
- net CS: track 20.1 -> 6.93 mm, vias 0 -> 1
- net GP15: track 0.00 -> 12.6 mm, vias 0 -> 1
- net D2: track 14.3 -> 2.32 mm
- net GP2: track 0.00 -> 11.6 mm, vias 0 -> 1
- net 5V: track 17.9 -> 29.4 mm
- net GP14: track 0.00 -> 11.5 mm, vias 0 -> 1
- net D3: track 3.68 -> 15.0 mm
- net GP9: track 0.00 -> 10.1 mm
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Other:
- board size 18 x 33 mm -> 18 x 33.2 mm
- board text added: "BOOT"
- board text added: "rev 0.1"
