File: Pro_Smolcro/Pro_Smolcro.kicad_sch (KiCad schematic)
At the start: 30 parts, among them J1 SHOU HAN TYPE-C 16PIN 2MD(073), SW1 BOOT, U1 RP2040, U2 TLV1117LV33DCYR, U3 W25Q128JVS, Y1 ABM8-272-T3

Commit message: finished layout of the main components
Parts:
- removed LeftSide, RightSide: Conn_01x12, Connector_PinSocket_2.54mm:PinSocket_1x12_P2.54mm_Vertical, symbol Connector_Generic:Conn_01x12
- removed U2: TLV1117LV33DCYR, Package_TO_SOT_SMD:SOT-223-3_TabPin2, symbol Regulator_Linear:TLV1117-33
- added J2: Conn_01x05, Connector_PinSocket_2.54mm:PinSocket_1x05_P2.54mm_Vertical, symbol Connector_Generic:Conn_01x05
- added J3, J4: Conn_01x13, Connector_PinSocket_2.54mm:PinSocket_1x13_P2.54mm_Vertical, symbol Connector_Generic:Conn_01x13
- added SW2: SW_Push, MyKeebLib:SW_TS-1088-AR02016, symbol Switch:SW_Push
- added U4: TLV75733PDBV, Package_TO_SOT_SMD:SOT-23-5, symbol Regulator_Linear:TLV75733PDBV
- C1, C11, C12, C2: footprint (none) -> Capacitor_SMD:C_0603_1608Metric
- C10, C13, C3, C4, C5, C6, C7, C8, C9: footprint (none) -> Capacitor_SMD:C_0402_1005Metric
- C14, C15: footprint (none) -> Capacitor_SMD:C_0402_1005Metric; LCSC (none) -> C86285
- R1, R2, R5, R6, R7: footprint (none) -> Resistor_SMD:R_0402_1005Metric
- R3, R4: footprint (none) -> Resistor_SMD:R_0402_1005Metric; LCSC (none) -> C2759791
- SW1: value BOOT -> SW_Push; footprint (none) -> MyKeebLib:SW_TS-1088-AR02016; LCSC (none) -> C720477
- U3: LCSC (none) -> C97521
- Y1: LCSC (none) -> C20625731
Connections:
- net +3V3: now also J4.5 (Pin_5), U4.5 (OUT); no longer U1.26 (RUN)
- net +5V: now also J4.2 (Pin_2), U4.1 (IN), U4.3 (EN)
- net GND: now also SW1.1, J3.4 (Pin_4), J3.5 (Pin_5), J4.3 (Pin_3), SW2.2, U4.2 (GND); no longer SW1.2
- net GP8: now reaches U1.11 (GPIO8)
- net GP8: now also J3.12 (Pin_12)
- net GP9: now reaches U1.12 (GPIO9)
- net GP9: now also J3.13 (Pin_13)
- net GP10: now reaches U1.13 (GPIO10)
- net GP10: now also J3.1 (Pin_1)
- net GP11: now reaches U1.14 (GPIO11)
- net GP11: now also J4.1 (Pin_1)
- net GP12: now reaches U1.15 (GPIO12)
- net GP12: now also J2.1 (Pin_1)
- net GP13: now reaches U1.16 (GPIO13)
- net GP13: now also J2.2 (Pin_2)
- net GP14: now reaches U1.17 (GPIO14)
- net GP14: now also J2.3 (Pin_3)
- net GP15: now reaches U1.18 (GPIO15)
- net GP15: now also J2.4 (Pin_4)
- net GP0: now reaches U1.2 (GPIO0)
- net GP0: now also J3.2 (Pin_2)
- net GP16: now reaches U1.27 (GPIO16)
- net GP16: now also J2.5 (Pin_5)
- net GP1: now reaches U1.3 (GPIO1)
- net GP1: now also J3.3 (Pin_3)
- net GP20: now reaches U1.31 (GPIO20)
- net GP20: now also J4.11 (Pin_11)
- net GP21: now reaches U1.32 (GPIO21)
- net GP21: now also J4.13 (Pin_13)
- net GP22: now reaches U1.34 (GPIO22)
- net GP22: now also J4.10 (Pin_10)
- net GP23: now reaches U1.35 (GPIO23)
- net GP23: now also J4.12 (Pin_12)
- net GP26: now reaches U1.38 (GPIO26_ADC0)
- net GP26: now also J4.9 (Pin_9)
- net GP27: now reaches U1.39 (GPIO27_ADC1)
- net GP27: now also J4.8 (Pin_8)
- net GP2: now reaches U1.4 (GPIO2)
- net GP2: now also J3.6 (Pin_6)
- net GP28: now reaches U1.40 (GPIO28_ADC2)
- net GP28: now also J4.7 (Pin_7)
- net GP29: now reaches U1.41 (GPIO29_ADC3)
- net GP29: now also J4.6 (Pin_6)
- net USBN: now reaches R4.2, U1.46 (USB_DM)
- net USBP: now reaches R3.2, U1.47 (USB_DP)
- net GP3: now reaches U1.5 (GPIO3)
- net GP3: now also J3.7 (Pin_7)
- net GP4: now reaches U1.6 (GPIO4)
- net GP4: now also J3.8 (Pin_8)
- net GP5: now reaches U1.7 (GPIO5)
- net GP5: now also J3.9 (Pin_9)
- net GP6: now reaches U1.8 (GPIO6)
- net GP6: now also J3.10 (Pin_10)
- net GP7: now reaches U1.9 (GPIO7)
- net GP7: now also J3.11 (Pin_11)
- net at R6.1: now also SW2.1; no longer SW1.1
- new net RST: J4.4 (Pin_4), SW1.2, U1.26 (RUN)
- no-connect marks 2 -> 9
Other:
- note added: "If you pull reset pin to ground the controller will restart"
- note added: "Pinout"
- moved on the sheet: R3, R4

Commit message: finished the layout
Parts:
- added D4: LED, LED_SMD:LED_0402_1005Metric, symbol Device:LED
- added R8: 68R, Resistor_SMD:R_0402_1005Metric, symbol Device:R
- added TP4, TP5: TestPoint, TestPoint:TestPoint_Pad_1.0x1.0mm, symbol Connector:TestPoint
- R5: now left out of the parts list
- R6, SW1, SW2: now not fitted; now left out of the parts list
Connections:
- net +3V3: now also R8.1
- net CS: now also TP4.1
- net GND: now also U4.4 (GNDNC), D4.1 (K), TP5.1
- net GNDNC: now reaches U4.4 (GNDNC)
- new net: D4.2 (A), R8.2
Other:
- note added: "Test points used instead of a button :D (no space unfortunatly)"
